File: FMC-board/development-prototype/FMC_prototype.sch (EAGLE design)
At the start: 72 parts, among them U1 TPS79301, U2 TPS79333, U3 ADN4663, U4 ADN4663, U5 ADN4664, U6 PDS1-S12-S5-S, U7 TPS79301

Commit message: More routing.
Connections:
- removed net CS_ISO: DO_ISO.VOA, U4.DIN1
- removed net H17: DO_ISO.VID, FMCG$1.P$17
- new net CS_IS0: DO_ISO.VOB, U4.DIN1
- new net H13: DO_ISO.VIA, FMCG$1.P$13
- new net H17_ISO: DO_ISO.VOA, G22_ISO.1
- new net H22_ISO: DI_ISO.VIB, H22_ISO.1
- new net H23_ISO: DI_ISO.VIA, H21_ISO.1
- net CS: now also DO_ISO.VIB, FMCG$1.P$14; no longer DO_ISO.VIA, FMCG$1.P$13
- net MISO1_ISO: now also DI_ISO.VID; no longer DI_ISO.VIB
- net MISO2_ISO: now also DI_ISO.VIC; no longer DI_ISO.VIA
- net MOSI: now also DO_ISO.VID, FMCG$1.P$17; no longer DO_ISO.VIC, FMCG$1.P$16
- net MOSI_ISO: now also DO_ISO.VOD; no longer DO_ISO.VOC
- net SCLK: now also DO_ISO.VIC, FMCG$1.P$16; no longer DO_ISO.VIB, FMCG$1.P$14
- net SCLK_ISO: now also DO_ISO.VOC; no longer DO_ISO.VOB
Changed lines of the file:
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@@
 <segment>
 <pinref part="U5" gate="G$1" pin="ROUT1"/>
-<pinref part="DI_ISO" gate="G$1" pin="VIA"/>
 <wire x1="177.8" y1="195.58" x2="182.88" y2="195.58" width="0.1524" layer="91"/>
-<wire x1="182.88" y1="195.58" x2="182.88" y2="175.26" width="0.1524" layer="91"/>
-<wire x1="182.88" y1="175.26" x2="210.82" y2="175.26" width="0.1524" layer="91"/>
-<label x="195.58" y="175.26" size="1.778" layer="95"/>
+<wire x1="182.88" y1="195.58" x2="182.88" y2="170.18" width="0.1524" layer="91"/>
+<pinref part="DI_ISO" gate="G$1" pin="VIC"/>
+<wire x1="210.82" y1="170.18" x2="182.88" y2="170.18" width="0.1524" layer="91"/>
+<label x="195.58" y="170.18" size="1.778" layer="95"/>
 </segment>
 </net>
@@
 <segment>
 <pinref part="U5" gate="G$1" pin="ROUT2"/>
-<wire x1="210.82" y1="172.72" x2="180.34" y2="172.72" width="0.1524" layer="91"/>
-<wire x1="180.34" y1="172.72" x2="180.34" y2="190.5" width="0.1524" layer="91"/>
+<wire x1="180.34" y1="167.64" x2="180.34" y2="190.5" width="0.1524" layer="91"/>
 <wire x1="180.34" y1="190.5" x2="177.8" y2="190.5" width="0.1524" layer="91"/>
-<pinref part="DI_ISO" gate="G$1" pin="VIB"/>
-<label x="195.58" y="172.72" size="1.778" layer="95"/>
+<pinref part="DI_ISO" gate="G$1" pin="VID"/>
+<wire x1="210.82" y1="167.64" x2="180.34" y2="167.64" width="0.1524" layer="91"/>
+<label x="195.58" y="167.64" size="1.778" layer="95"/>
 </segment>
 </net>
@@
 <net name="MOSI_ISO" class="0">
 <segment>
+<pinref part="DO_ISO" gate="G$1" pin="VOD"/>
+<label x="195.58" y="142.24" size="1.778" layer="95"/>
 <pinref part="U3" gate="G$1" pin="DIN2"/>
 <wire x1="180.34" y1="147.32" x2="177.8" y2="147.32" width="0.1524" layer="91"/>
-<wire x1="180.34" y1="139.7" x2="180.34" y2="147.32" width="0.1524" layer="91"/>
-<pinref part="DO_ISO" gate="G$1" pin="VOC"/>
-<wire x1="180.34" y1="139.7" x2="210.82" y2="139.7" width="0.1524" layer="91"/>
-<label x="195.58" y="139.7" size="1.778" layer="95"/>
-</segment>
-</net>
-<net name="CS_ISO" class="0">
-<segment>
-<wire x1="185.42" y1="134.62" x2="185.42" y2="109.22" width="0.1524" layer="91"/>
-<wire x1="185.42" y1="109.22" x2="177.8" y2="109.22" width="0.1524" layer="91"/>
-<pinref part="U4" gate="G$1" pin="DIN1"/>
-<pinref part="DO_ISO" gate="G$1" pin="VOA"/>
-<wire x1="210.82" y1="134.62" x2="185.42" y2="134.62" width="0.1524" layer="91"/>
-<label x="195.58" y="134.62" size="1.778" layer="95"/>
+<wire x1="210.82" y1="142.24" x2="180.34" y2="142.24" width="0.1524" layer="91"/>
+<wire x1="180.34" y1="142.24" x2="180.34" y2="147.32" width="0.1524" layer="91"/>
 </segment>
 </net>
@@
 <net name="SCLK_ISO" class="0">
 <segment>
+<pinref part="DO_ISO" gate="G$1" pin="VOC"/>
+<label x="195.58" y="139.7" size="1.778" layer="95"/>
+<wire x1="182.88" y1="139.7" x2="210.82" y2="139.7" width="0.1524" layer="91"/>
 <wire x1="177.8" y1="152.4" x2="182.88" y2="152.4" width="0.1524" layer="91"/>
-<wire x1="182.88" y1="152.4" x2="182.88" y2="137.16" width="0.1524" layer="91"/>
 <pinref part="U3" gate="G$1" pin="DIN1"/>
-<pinref part="DO_ISO" gate="G$1" pin="VOB"/>
-<wire x1="182.88" y1="137.16" x2="210.82" y2="137.16" width="0.1524" layer="91"/>
-<label x="195.58" y="137.16" size="1.778" layer="95"/>
+<wire x1="182.88" y1="152.4" x2="182.88" y2="139.7" width="0.1524" layer="91"/>
 </segment>
 </net>
@@
 <net name="MOSI" class="0">
 <segment>
+<pinref part="DO_ISO" gate="G$1" pin="VID"/>
+<wire x1="246.38" y1="142.24" x2="256.54" y2="142.24" width="0.1524" layer="91"/>
+<label x="246.38" y="142.24" size="1.778" layer="95"/>
+</segment>
+<segment>
+<pinref part="FMC" gate="G$1" pin="P$17"/>
+<wire x1="393.7" y1="264.16" x2="381" y2="264.16" width="0.1524" layer="91"/>
+<label x="381" y="264.16" size="1.778" layer="95"/>
+</segment>
+</net>
+<net name="SCLK" class="0">
+<segment>
+<pinref part="DO_ISO" gate="G$1" pin="VIC"/>
+<wire x1="256.54" y1="139.7" x2="246.38" y2="139.7" width="0.1524" layer="91"/>
+<label x="246.38" y="139.7" size="1.778" layer="95"/>
+</segment>
+<segment>
 <pinref part="FMC" gate="G$1" pin="P$16"/>
 <wire x1="393.7" y1="266.7" x2="381" y2="266.7" width="0.1524" layer="91"/>
 <label x="381" y="266.7" size="1.778" layer="95"/>
 </segment>
-<segment>
-<pinref part="DO_ISO" gate="G$1" pin="VIC"/>
-<wire x1="256.54" y1="139.7" x2="246.38" y2="139.7" width="0.1524" layer="91"/>
-<label x="246.38" y="139.7" size="1.778" layer="95"/>
-</segment>
-</net>
-<net name="SCLK" class="0">
+</net>
+<net name="CS" class="0">
+<segment>
+<pinref part="DO_ISO" gate="G$1" pin="VIB"/>
+<wire x1="246.38" y1="137.16" x2="256.54" y2="137.16" width="0.1524" layer="91"/>
+<label x="246.38" y="137.16" size="1.778" layer="95"/>
+</segment>
 <segment>
 <pinref part="FMC" gate="G$1" pin="P$14"/>
@@
 <label x="381" y="271.78" size="1.778" layer="95"/>
 </segment>
-<segment>
-<pinref part="DO_ISO" gate="G$1" pin="VIB"/>
-<wire x1="246.38" y1="137.16" x2="256.54" y2="137.16" width="0.1524" layer="91"/>
-<label x="246.38" y="137.16" size="1.778" layer="95"/>
-</segment>
-</net>
-<net name="CS" class="0">
+</net>
+<net name="N$9" class="0">
+<segment>
+<pinref part="FMC" gate="G$1" pin="P$76"/>
+<wire x1="444.5" y1="215.9" x2="441.96" y2="215.9" width="0.1524" layer="91"/>
+</segment>
+</net>
+<net name="H23" class="0">
+<segment>
+<pinref part="FMC" gate="G$1" pin="P$23"/>
+<wire x1="393.7" y1="248.92" x2="381" y2="248.92" width="0.1524" layer="91"/>
+<label x="381" y="248.92" size="1.778" layer="95"/>
+</segment>
+<segment>
+<pinref part="DI_ISO" gate="G$1" pin="VOA"/>
+<wire x1="246.38" y1="175.26" x2="261.62" y2="175.26" width="0.1524" layer="91"/>
+<label x="248.92" y="175.26" size="1.778" layer="95"/>
+</segment>
+</net>
+<net name="H22" class="0">
+<segment>
+<pinref part="FMC" gate="G$1" pin="P$22"/>
+<wire x1="393.7" y1="251.46" x2="381" y2="251.46" width="0.1524" layer="91"/>
+<label x="381" y="251.46" size="1.778" layer="95"/>
+</segment>
+<segment>
+<pinref part="DI_ISO" gate="G$1" pin="VOB"/>
+<wire x1="246.38" y1="172.72" x2="261.62" y2="172.72" width="0.1524" layer="91"/>
+<label x="248.92" y="172.72" size="1.778" layer="95"/>
+</segment>
+</net>
+<net name="H13" class="0">
 <segment>
 <pinref part="DO_ISO" gate="G$1" pin="VIA"/>
@@
 </segment>
 </net>
-<net name="N$9" class="0">
-<segment>
-<pinref part="FMC" gate="G$1" pin="P$76"/>
-<wire x1="444.5" y1="215.9" x2="441.96" y2="215.9" width="0.1524" layer="91"/>
-</segment>
-</net>
-<net name="H23" class="0">
-<segment>
-<pinref part="FMC" gate="G$1" pin="P$23"/>
-<wire x1="393.7" y1="248.92" x2="381" y2="248.92" width="0.1524" layer="91"/>
-<label x="381" y="248.92" size="1.778" layer="95"/>
-</segment>
-<segment>
-<pinref part="DI_ISO" gate="G$1" pin="VOA"/>
-<wire x1="246.38" y1="175.26" x2="261.62" y2="175.26" width="0.1524" layer="91"/>
-<label x="248.92" y="175.26" size="1.778" layer="95"/>
-</segment>
-</net>
-<net name="H22" class="0">
-<segment>
-<pinref part="FMC" gate="G$1" pin="P$22"/>
-<wire x1="393.7" y1="251.46" x2="381" y2="251.46" width="0.1524" layer="91"/>
-<label x="381" y="251.46" size="1.778" layer="95"/>
-</segment>
-<segment>
-<pinref part="DI_ISO" gate="G$1" pin="VOB"/>
-<wire x1="246.38" y1="172.72" x2="261.62" y2="172.72" width="0.1524" layer="91"/>
-<label x="248.92" y="172.72" size="1.778" layer="95"/>
-</segment>
-</net>
-<net name="H17" class="0">
-<segment>
-<pinref part="FMC" gate="G$1" pin="P$17"/>
-<wire x1="393.7" y1="264.16" x2="381" y2="264.16" width="0.1524" layer="91"/>
-<label x="381" y="264.16" size="1.778" layer="95"/>
-</segment>
-<segment>
-<pinref part="DO_ISO" gate="G$1" pin="VID"/>
-<wire x1="246.38" y1="142.24" x2="256.54" y2="142.24" width="0.1524" layer="91"/>
-<label x="246.38" y="142.24" size="1.778" layer="95"/>
-</segment>
-</net>
+<net name="H17_ISO" class="0">
+<segment>
+<pinref part="G22_ISO" gate="G$1" pin="1"/>
+<wire x1="68.58" y1="78.74" x2="83.82" y2="78.74" width="0.1524" layer="91"/>
+<label x="68.58" y="78.74" size="1.778" layer="95"/>
+</segment>
+<segment>
+<pinref part="DO_ISO" gate="G$1" pin="VOA"/>
+<wire x1="210.82" y1="134.62" x2="195.58" y2="134.62" width="0.1524" layer="91"/>
+<label x="195.58" y="134.62" size="1.778" layer="95"/>
+</segment>
+</net>
+<net name="H22_ISO" class="0">
+<segment>
+<pinref part="DI_ISO" gate="G$1" pin="VIB"/>
+<wire x1="210.82" y1="172.72" x2="195.58" y2="172.72" width="0.1524" layer="91"/>
+<label x="195.58" y="172.72" size="1.778" layer="95"/>
+</segment>
+<segment>
+<pinref part="H22_ISO" gate="G$1" pin="1"/>
+<wire x1="68.58" y1="99.06" x2="83.82" y2="99.06" width="0.1524" layer="91"/>
+<label x="68.58" y="99.06" size="1.778" layer="95"/>
+</segment>
+</net>
+<net name="H23_ISO" class="0">
+<segment>
+<pinref part="DI_ISO" gate="G$1" pin="VIA"/>
+<wire x1="210.82" y1="175.26" x2="198.12" y2="175.26" width="0.1524" layer="91"/>
+<wire x1="195.58" y1="175.26" x2="198.12" y2="175.26" width="0.1524" layer="91"/>
+<label x="195.58" y="175.26" size="1.778" layer="95"/>
+</segment>
+<segment>
+<pinref part="H21_ISO" gate="G$1" pin="1"/>
+<wire x1="68.58" y1="119.38" x2="83.82" y2="119.38" width="0.1524" layer="91"/>
+<label x="68.58" y="119.38" size="1.778" layer="95"/>
+</segment>
+</net>
+<net name="CS_IS0" class="0">
+<segment>
+<pinref part="DO_ISO" gate="G$1" pin="VOB"/>
+<wire x1="182.88" y1="137.16" x2="210.82" y2="137.16" width="0.1524" layer="91"/>
+<label x="195.58" y="137.16" size="1.778" layer="95"/>
+<pinref part="U4" gate="G$1" pin="DIN1"/>
+<wire x1="182.88" y1="109.22" x2="177.8" y2="109.22" width="0.1524" layer="91"/>
+<wire x1="182.88" y1="137.16" x2="182.88" y2="109.22" width="0.1524" layer="91"/>
+</segment>
+</net>

Commit message: Nearly finished with routing, try to finish tonight.
Parts:
- removed C16: 1.0u, RHD2000_eval_board:C_0805
- removed C19: 10n, RHD2000_eval_board:C_0603
- removed C25: 15p, RHD2000_eval_board:C_0603
- removed C26: 22u, RHD2000_eval_board:C_1206
- removed D3: SML-D1, jonnew:LED_0603
- removed LINK-5V, LINK_GNDS: (no value), jumper:JP2E
- removed R12: 820, RHD2000_eval_board:R_0603
- removed R8: 95.3k, RHD2000_eval_board:R_0603
- removed R9: 30.9k, RHD2000_eval_board:R_0603
- removed U7: TPS79301, RHD2000_eval_board:TPS79301
- added +4.5V: TPPAD1-17, testpad:TPPAD1-17
- added C21, C40: 10uF, puggleboard:C_1206
- added C33: 1nF, puggleboard:C_0603
- added C35, C37: 10nF, puggleboard:C_0603
- added L2: MPZ1608, puggleboard:L_0603
- added LINK-5V1: (no value), jumper:JP2E
- added R16: 13.7k, puggleboard:R_0603
- added R17: 4.7k, puggleboard:R_0603
- added U8: 4901, puggleboard:TPS7A4901DGNR
- renumbered G22_ISO to H13, H21_ISO to H23, H22_ISO to H14
Connections:
- removed net +5V0_EXT: L1.1, LINK-5V.2
- removed net CS_IS0: DO_ISO.VOB, U4.DIN1
- removed net H17_ISO: DO_ISO.VOA, H13.1
- removed net H22: DI_ISO.VOB, FMCG$1.P$22
- removed net H22_ISO: DI_ISO.VIB, H14.1
- removed net MOSI+_ISOLATED: A_ISOLATED.MOSI+, U3.DOUT2+
- removed net MOSI-_ISOLATED: A_ISOLATED.MOSI-, U3.DOUT2-
- removed net N$14: C19.1, U7.NR
- removed net N$27: C25.2, R8.1, R9.1, U7.FB
- removed net N$4: D3.A, R12.2
- removed net SCLK+_ISOLATED: A_ISOLATED.SCLK+, U3.DOUT1+
- removed net SCLK-_ISOLATED: A_ISOLATED.SCLK-, U3.DOUT1-
- new net +4.5V: +4.5V.TP, C37.1, C40.1, R16.1, U8.OUT
- new net AGND1: C37.2, R16.2, R17.1, U8.FB
- new net CS_ISO: DO_ISO.VOC, U4.DIN1
- new net GND1: C21.2, C33.2, C35.2, C40.2, R17.2, U8.EP, U8.GND
- new net H13_ISO: DI_ISO.VID, H13.1
- new net H14: DI_ISO.VOC, FMCG$1.P$14
- new net H14_ISO: DI_ISO.VIC, H14.1
- new net N$1: C35.1, U8.NR/SS
- new net N$12: A_ISOLATED.MOSI+, U3.DOUT1+
- new net N$13: A_ISOLATED.MOSI-, U3.DOUT1-
- new net N$15: A_ISOLATED.SCLK+, U3.DOUT2+
- new net N$16: A_ISOLATED.SCLK-, U3.DOUT2-
- new net N$3: D4.C, LINK-5V1.1, U$4.S
- new net VDD_POST_LC: C21.1, C33.1, L2.2, U8.EN, U8.IN
- net +3V6: no longer C25.1, C26.1, R12.1, R8.2, U7.OUT
- net +5V0_ISO-PRE: now also L1.1; no longer LINK-5V.3
- net 12V_FPGA: now also LINK-5V1.3
- net AUX_VDD: now also L2.1, LINK-5V1.2; no longer C16.1, D4.C, LINK-5V.1, U$4.S, U7.EN, U7.IN
- net CS: now also DO_ISO.VIC, FMCG$1.P$22; no longer DO_ISO.VIB, FMCG$1.P$14
- net GND: no longer C16.2, C19.2, C26.2, D3.C, LINK_GNDS.3, R9.2, U7.GND
- net GND_ISO: no longer LINK_GNDS.2
- net H13: now also DI_ISO.VOD; no longer DO_ISO.VIA
- net H23: now also DO_ISO.VID; no longer DI_ISO.VOA
- net H23_ISO: now also DO_ISO.VOD; no longer DI_ISO.VIA
- net MISO1: now also DI_ISO.VOA, FMCG$1.P$17; no longer DI_ISO.VOD, FMCG$1.P$19
- net MISO1+_ISOLATED: now also U5.RIN1+; no longer U5.RIN2+
- net MISO1-_ISOLATED: now also U5.RIN1-; no longer U5.RIN2-
- net MISO1_ISO: now also DI_ISO.VIA, U5.ROUT1; no longer DI_ISO.VID, U5.ROUT2
- net MISO2: now also DI_ISO.VOB, FMCG$1.P$16; no longer DI_ISO.VOC, FMCG$1.P$20
- net MISO2+_ISOLATED: now also U5.RIN2+; no longer U5.RIN1+
- net MISO2-_ISOLATED: now also U5.RIN2-; no longer U5.RIN1-
- net MISO2_ISO: now also DI_ISO.VIB, U5.ROUT2; no longer DI_ISO.VIC, U5.ROUT1
- net MOSI: now also DO_ISO.VIA, FMCG$1.P$19; no longer DO_ISO.VID, FMCG$1.P$17
- net MOSI_ISO: now also DO_ISO.VOA, U3.DIN1; no longer DO_ISO.VOD, U3.DIN2
- net SCLK: now also DO_ISO.VIB, FMCG$1.P$20; no longer DO_ISO.VIC, FMCG$1.P$16
- net SCLK_ISO: now also DO_ISO.VOB, U3.DIN2; no longer DO_ISO.VOC, U3.DIN1
Other:
- moved on the sheet: C7, U3

Commit message: Hard routing complete
- Inner SMAs need hookups
- Should bezel be tied to GND_ISO?
- Re-add testpoints (pad style)
- Silkscreen...
Parts:
- removed +4.5V: TPPAD1-17, testpad:TPPAD1-17
- removed TP_C10, TP_C11: 142-0701, jonnew:COAX_SMA-VERT
- added C16: 1nF, jonnew:C_0603
- C1: value 22u -> 10uF; device RHD2000_eval_board:C_1206 -> puggleboard:C_1206
- C2: value 15p -> 10uF; device RHD2000_eval_board:C_0603 -> puggleboard:C_1206
- C33, C35, C37: device puggleboard:C_0603 -> jonnew:C_0603
- C4: value 10n -> 10nF; device RHD2000_eval_board:C_0603 -> jonnew:C_0603
- C9: value 1.0u -> 10nF; device RHD2000_eval_board:C_0805 -> jonnew:C_0603
- L2: device puggleboard:L_0603 -> jonnew:L_0603
- R1: value 820 -> 20k; device RHD2000_eval_board:R_0603 -> jonnew:R_0603
- R16: value 13.7k -> 20k; device puggleboard:R_0603 -> jonnew:R_0603
- R17: value 4.7k -> 10k; device puggleboard:R_0603 -> jonnew:R_0603
- R5: value 95.3k -> 10k; device RHD2000_eval_board:R_0603 -> jonnew:R_0603
- R6: value 30.9k -> 820
- U1: value TPS79301 -> 4901; device RHD2000_eval_board:TPS79301 -> puggleboard:TPS7A4901DGNR
Connections:
- removed net +4.5V: +4.5V.TP, C37.1, C40.1, R16.1, U8.OUT
- removed net GND1: C21.2, C33.2, C35.2, C40.2, R17.2, U8.EP, U8.GND
- removed net N$11: R1.2, U$32.A
- removed net N$36: C4.1, U1.NR
- removed net N$37: C2.2, R5.1, R6.1, U1.FB
- new net AGND2: C4.2, R1.2, R5.1, U1.FB
- new net N$4: C9.1, U1.NR/SS
- new net N$8: R6.2, U$32.A
- net +3V6: now also C37.1, C40.1, R16.1, U8.OUT
- net +3V6_ISO: now also C4.1, R6.1; no longer C1.1, R5.2
- net +5V0_ISO: now also C1.1, C16.1; no longer C9.1
- net GND: now also C21.2, C33.2, C35.2, C40.2, R17.2, U8.EP, U8.GND; no longer TP_C10.2, TP_C11.2
- net GND_ISO: now also C16.2, C2.2, R5.2, U1.EP; no longer C4.2, R6.2
Other:
- moved on the sheet: C1, C2, C4, C9, L1, R1, R5, R6, U$32
